Commit message: Switch to effort joints and 4 casters

File: robots/active_caster.xacro (robot description, xacro)
@@ -3,4 +3,5 @@
   <xacro:include filename="../urdf/materials/materials.xacro"/>
   <xacro:include filename="../urdf/utils.urdf.xacro"/>
+  <xacro:include filename="../urdf/plugins.gazebo.xacro"/>
   <!-- Set up definitions of parts of robot body -->
   <xacro:include filename="../urdf/base/active_caster_base.urdf.xacro"/>

File: urdf/base/active_caster_base.urdf.xacro (robot description, xacro)
@@ -2,4 +2,5 @@
 <!-- Dyno active caster base -->
 <robot xmlns:xacro="http://ros.org/wiki/xacro">
+  <xacro:include filename="active_caster_base.gazebo.xacro"/>
   <xacro:include filename="../wheels/active_caster/active_caster.urdf.xacro"/>
   <!-- Active caster characteristics -->
@@ -9,4 +10,21 @@
   <xacro:macro name="base">
     <link name="base_link">
+      <visual>
+        <origin xyz="0.2 0 0" rpy="0 ${M_PI/2} 0"/>
+        <geometry>
+          <cylinder length="0.02" radius="0.01"/>
+        </geometry>
+      </visual>
+      <collision>
+        <origin xyz="0 0 0.2" rpy="0 0 0"/>
+        <geometry>
+          <cylinder length="0.1" radius="0.2"/>
+        </geometry>
+      </collision>
+      <inertial>
+        <origin xyz="0 0 0" rpy="0 0 0"/>
+        <mass value="10.0"/>
+        <box_inertia m="10.0" x="0.3" y="0.3" z="0.1"/>
+      </inertial>
     </link>
     <!-- Base footprint -->
@@ -18,7 +36,17 @@
     </joint>
     <!-- Macros -->
+    <!-- Triangle -->
+    <!--
     <active_caster name="fl_caster" parent="base_link" x_offset="${wheel_separation/(sqrt(3)*2)}" y_offset="${wheel_separation/2}"/>
     <active_caster name="fr_caster" parent="base_link" x_offset="${wheel_separation/(sqrt(3)*2)}" y_offset="${-wheel_separation/2}"/>
     <active_caster name="rc_caster" parent="base_link" x_offset="${-wheel_separation/sqrt(3)}" y_offset="0"/>
+    -->
+    <!-- Square -->
+    <active_caster name="fl_caster" parent="base_link" x_offset="${wheel_separation/2}" y_offset="${wheel_separation/2}"/>
+    <active_caster name="fr_caster" parent="base_link" x_offset="${wheel_separation/2}" y_offset="${-wheel_separation/2}"/>
+    <active_caster name="rl_caster" parent="base_link" x_offset="${-wheel_separation/2}" y_offset="${wheel_separation/2}"/>
+    <active_caster name="rr_caster" parent="base_link" x_offset="${-wheel_separation/2}" y_offset="${-wheel_separation/2}"/>
+    <!-- Gazebo -->
+    <base_gazebo/>
   </xacro:macro>
 </robot>

File: urdf/wheels/active_caster/active_caster.gazebo.xacro (robot description, xacro)
@@ -1,7 +1,7 @@
 <?xml version="1.0"?>
 <robot xmlns:xacro="http://ros.org/wiki/xacro">
-  <xacro:macro name="drive_wheel_gazebo" params="name">
+  <xacro:macro name="wheel_gazebo" params="name">
     <!-- Contact model for the wheel surface -->
-   <gazebo reference="${name}_link">
+   <gazebo reference="${name}">
      <!--
      <kp>0.1</kp>
@@ -14,5 +14,5 @@
      <fdir1>1 0 0</fdir1>
      <maxVel>1.0</maxVel>
-     <minDepth>0.003</minDepth>
+     <minDepth>0.001</minDepth>
      <implicitSpringDamper>1</implicitSpringDamper>
      <material>Gazebo/DarkGrey</material>

File: urdf/wheels/active_caster/active_caster.urdf.xacro (robot description, xacro)
@@ -1,12 +1,33 @@
 <?xml version="1.0"?>
 <robot xmlns:xacro="http://ros.org/wiki/xacro">
+  <xacro:include filename="active_caster.gazebo.xacro"/>
   <xacro:macro name="active_caster" params="name x_offset y_offset parent">
     <xacro:property name="wheel_radius" value="0.02"/>
     <xacro:property name="wheel_width" value="0.015"/>
     <xacro:property name="wheel_mass" value="0.1"/>
-    <xacro:property name="x_yoke_offset" value="-0.0676"/>
+    <xacro:property name="x_yoke_offset" value="-0.04"/>
     <xacro:property name="z_yoke_offset" value="-0.034"/>
     <!-- Mount -->
-    <link name="${name}_mount_link"/>
+    <link name="${name}_mount_link">
+      <!--
+      <visual>
+        <origin xyz="0 0 0" rpy="0 0 0"/>
+        <geometry>
+          <cylinder length="0.001" radius="0.001"/>
+        </geometry>
+      </visual>
+       -->
+      <collision>
+        <origin xyz="0 0 0" rpy="0 0 0"/>
+        <geometry>
+          <cylinder length="0.01" radius="0.01"/>
+        </geometry>
+      </collision>
+      <inertial>
+        <origin xyz="0 0 0" rpy="0 0 0"/>
+        <mass value="0.1"/>
+        <box_inertia m="0.1" x="0.1" y="0.1" z="0.1"/>
+      </inertial>
+    </link>
     <joint name="${name}_mount_joint" type="fixed">
       <origin xyz="${x_offset} ${y_offset} 0" rpy="0 0 0"/>
@@ -19,8 +40,19 @@
         <origin xyz="0 0 0" rpy="0 0 0"/>
         <geometry>
-          <cylinder length="0.01" radius="0.0387"/>
+          <cylinder length="0.01" radius="0.03"/>
         </geometry>
         <material name="blue"/>
       </visual>
+      <collision>
+        <origin xyz="0 0 0" rpy="0 0 0"/>
+        <geometry>
+          <cylinder length="0.01" radius="0.01"/>
+        </geometry>
+      </collision>
+      <inertial>
+        <origin xyz="0 0 0" rpy="0 0 0"/>
+        <mass value="0.1"/>
+        <box_inertia m="0.1" x="0.1" y="0.1" z="0.1"/>
+      </inertial>
     </link>
     <joint name="${name}_steer_joint" type="continuous">
@@ -39,4 +71,16 @@
         <material name="orange"/>
       </visual>
+      <collision>
+        <origin xyz="0 0 0" rpy="0 0 0"/>
+        <geometry>
+          <cylinder length="${wheel_width}" radius="${wheel_radius}"/>
+        </geometry>
+        <material name="orange"/>
+      </collision>
+      <inertial>
+        <origin xyz="0 0 0" rpy="0 0 0"/>
+        <mass value="0.5"/>
+        <cylinder_inertia m="0.5" r="${wheel_radius}" h="${wheel_width}"/>
+      </inertial>
     </link>
     <joint name="${name}_wheel_joint" type="continuous">
@@ -48,6 +92,8 @@
     </joint>
     <!-- Transmission -->
-    <xacro:simple_transmission name="${name}_steer_joint" interface="PositionJointInterface"/>
-    <xacro:simple_transmission name="${name}_wheel_joint" interface="VelocityJointInterface"/>
+    <xacro:simple_transmission name="${name}_steer_joint" interface="EffortJointInterface"/>
+    <xacro:simple_transmission name="${name}_wheel_joint" interface="EffortJointInterface"/>
+    <!-- Gazebo -->
+    <wheel_gazebo name="${name}_wheel_link"/>
   </xacro:macro>
 </robot>
